File: hardware/0.1/fx3-usb-misc.kicad_sch (KiCad schematic)
At the start: 21 parts

Commit message: first pass schematic done
Parts:
- added unit 2 of U301
- C301, C302, C305, C306: renamed from C?; footprint (none) -> Capacitor_SMD:C_0402_1005Metric; LCSC (none) -> C307331; MPN (none) -> CL05B104KB54PNC; Manufacturer (none) -> Samsung Electro-Mechanics
- C303, C304: renamed from C?; footprint (none) -> Capacitor_SMD:C_0402_1005Metric; Digikey (none) -> 490-8079-1-ND; LCSC (none) -> C2167421; MPN (none) -> GJM1555C1H130GB01D; Manufacturer (none) -> Murata Electronics
- R301, R306, R308: renamed from R?; footprint (none) -> Resistor_SMD:R_0402_1005Metric; LCSC (none) -> C60490; MPN (none) -> RC0402FR-0710KL; Manufacturer (none) -> Yageo
- R302: renamed from R?; footprint (none) -> Resistor_SMD:R_0402_1005Metric; LCSC (none) -> C114764; MPN (none) -> RC0402FR-07200RL; Manufacturer (none) -> Yageo
- R303: renamed from R?; footprint (none) -> Resistor_SMD:R_0402_1005Metric; LCSC (none) -> C144739; MPN (none) -> AC0402FR-076K04L; Manufacturer (none) -> Yageo
- R304, R305: renamed from R?; footprint (none) -> Resistor_SMD:R_0402_1005Metric; LCSC (none) -> C114762; MPN (none) -> RC0402FR-072K2L; Manufacturer (none) -> Yageo
- R307: renamed from R?; footprint (none) -> Resistor_SMD:R_0402_1005Metric; Manufacturer (none) -> Yageo
- U301: renamed from U?; footprint (none) -> josh-bga:BGA-121_10x10mm_Layout11x11_P0.8mm; Digikey (none) -> 448-CYUSB3014-BZXC-ND; LCSC (none) -> C462526; MPN (none) -> CYUSB3014-BZXC; Manufacturer (none) -> Cypress / Infineon
- U302: renamed from U?; LCSC (none) -> C115042; MPN (none) -> M24M02-DRMN6TP; Manufacturer (none) -> STMicroelectronics
- Y301: renamed from Y?; footprint (none) -> josh-oscillators:Crystal_SMD_2520-4Pin_2.5x2.0mm; Digikey (none) -> 644-1162-2-ND; MPN (none) -> EXS00A-CS05400; Manufacturer (none) -> NDK
Connections:
- net SDA: now reaches R305.2, U301.D10 (SDA_GPIO[59])
- net SDA: now also U302.5 (SDA); no longer U302.6 (SCL)
- net SCL: now reaches R304.2, U301.D9 (SCL_GPIO[58])
- net SCL: now also U302.6 (SCL); no longer U302.5 (SDA)
- no-connect marks 15 -> 28
Other:
- note added: "Bank 2 is unused"
- company: (none) -> Josh Johnson
- title: (none) -> Voyager Logic
- moved on the sheet: C301, C302, C303, C304, C305, C306, R301, R302, R303, R304, R305, R306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

Commit message: finalise BOM
Changed lines of the file:
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@@
   (symbol (lib_id "Device:C") (at 182.88 101.6 90) (unit 1)
     (in_bom yes) (on_board yes)
-    (property "Reference" "C306" (id 0) (at 186.69 100.33 90)
+    (property "Reference" "C306" (id 0) (at 189.23 100.33 90)
       (effects (font (size 1.27 1.27)) (justify left))
     )

Commit message: all components fit inside outline
Changed lines of the file:
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@@
   (symbol (lib_id "Device:C") (at 175.26 58.42 90) (unit 1)
     (in_bom yes) (on_board yes)
-    (property "Reference" "C304" (id 0) (at 177.8 57.15 90))
+    (property "Reference" "C304" (id 0) (at 179.07 57.15 90))
     (property "Value" "13p" (id 1) (at 178.435 59.69 90))
     (property "Footprint" "Capacitor_SMD:C_0402_1005Metric" (id 2) (at 179.07 57.4548 0)
@@
   (symbol (lib_id "Device:C") (at 175.26 47.625 90) (unit 1)
     (in_bom yes) (on_board yes)
-    (property "Reference" "C303" (id 0) (at 177.8 46.355 90))
+    (property "Reference" "C303" (id 0) (at 179.07 46.355 90))
     (property "Value" "13p" (id 1) (at 178.435 48.895 90))
     (property "Footprint" "Capacitor_SMD:C_0402_1005Metric" (id 2) (at 179.07 46.6598 0)

Commit message: break out bga
Parts:
- removed C301, C302: 100n, Capacitor_SMD:C_0402_1005Metric, symbol Device:C
- removed R301, R308: 10K, Resistor_SMD:R_0402_1005Metric, symbol Device:R
Connections:
- net GND: now also U301.B2 (FSLC[0]), U301.B4 (FSLC[1]), U301.E6 (FSLC[2])
- net USB3_TX_N: now also U301.A6 (SSTXM)
- net USB3_TX_P: now also U301.A5 (SSTXP)
- net at C304.1, U301.C7 (XTALOUT): now also Y301.3; no longer Y301.1
- net at C303.1, U301.C6 (XTALIN): now also Y301.1; no longer Y301.3
- net LED_B: no longer names the net of U301.E5 (GPIO[48])
- net LED_G: no longer names the net of U301.E1 (GPIO[47])
- net LED_R: no longer names the net of U301.F5 (GPIO[46])
- no-connect marks 28 -> 31
Other:
- note added: "Selects 19.2MHz Crystal"
- note removed: "0201 caps"

Commit message: erc = drc = 0, fixup BOM
Parts:
- R307: Manufacturer Yageo -> (none)
Changed lines of the file:
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@@
       (effects (font (size 1.27 1.27)) hide)
     )
-    (property "Manufacturer" "Yageo" (id 4) (at 43.815 161.29 0)
+    (property "Manufacturer" "" (id 4) (at 43.815 161.29 0)
       (effects (font (size 1.27 1.27)) hide)
     )

Commit message: component shortage changes
Parts:
- C303, C304: Digikey 490-8079-1-ND -> (none); LCSC C2167421 -> C2195053; MPN GJM1555C1H130GB01D -> GCM1555C1H130JA16D
Changed lines of the file:
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@@
       (effects (font (size 1.27 1.27)) hide)
     )
-    (property "Digikey" "490-8079-1-ND" (id 4) (at 175.26 58.42 0)
+    (property "Digikey" "" (id 4) (at 175.26 58.42 0)
       (effects (font (size 1.27 1.27)) hide)
     )
-    (property "LCSC" "C2167421" (id 5) (at 175.26 58.42 0)
+    (property "LCSC" "C2195053" (id 5) (at 175.26 58.42 0)
       (effects (font (size 1.27 1.27)) hide)
     )
-    (property "MPN" "GJM1555C1H130GB01D" (id 6) (at 175.26 58.42 0)
+    (property "MPN" "GCM1555C1H130JA16D" (id 6) (at 175.26 58.42 0)
       (effects (font (size 1.27 1.27)) hide)
     )
@@
       (effects (font (size 1.27 1.27)) hide)
     )
-    (property "Digikey" "490-8079-1-ND" (id 4) (at 175.26 47.625 0)
+    (property "Digikey" "" (id 4) (at 175.26 47.625 0)
       (effects (font (size 1.27 1.27)) hide)
     )
-    (property "LCSC" "C2167421" (id 5) (at 175.26 47.625 0)
+    (property "LCSC" "C2195053" (id 5) (at 175.26 47.625 0)
       (effects (font (size 1.27 1.27)) hide)
     )
-    (property "MPN" "GJM1555C1H130GB01D" (id 6) (at 175.26 47.625 0)
+    (property "MPN" "GCM1555C1H130JA16D" (id 6) (at 175.26 47.625 0)
       (effects (font (size 1.27 1.27)) hide)
     )
