File: hardware/0.1/usb-c.kicad_sch (KiCad schematic)
At the start: 32 parts, among them J201 USB_C_Receptacle, U201 USBLC6-2P6, U202 HD3SS3220, U203 TPD4EUSB30, U204 TPD4EUSB30

Commit message: usb 3 clean up
Connections:
- net RX1N renamed RX1_N
- net RX1P renamed RX1_P
- net RX2N renamed RX2_N
- net RX2P renamed RX2_P
- net TX1N renamed TX1_N
- net TX1P renamed TX1_P
- net TX2N renamed TX2_N
- net TX2P renamed TX2_P
Changed lines of the file:
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@@
     (effects (font (size 1.27 1.27)) (justify left bottom))
   )
-  (label "TX2N" (at 144.145 117.475 0)
+  (label "TX2_N" (at 144.145 117.475 0)
     (effects (font (size 1.27 1.27)) (justify left bottom))
   )
@@
     (effects (font (size 1.27 1.27)) (justify left bottom))
   )
-  (label "RX2P" (at 144.145 112.395 0)
+  (label "RX2_P" (at 144.145 112.395 0)
     (effects (font (size 1.27 1.27)) (justify left bottom))
   )
-  (label "RX2N" (at 144.145 109.855 0)
+  (label "RX2_N" (at 144.145 109.855 0)
     (effects (font (size 1.27 1.27)) (justify left bottom))
   )
-  (label "TX2P" (at 144.145 120.015 0)
+  (label "TX2_P" (at 144.145 120.015 0)
     (effects (font (size 1.27 1.27)) (justify left bottom))
   )
@@
     (effects (font (size 1.27 1.27)) (justify left bottom))
   )
-  (label "TX1P" (at 144.145 104.775 0)
+  (label "TX1_P" (at 144.145 104.775 0)
     (effects (font (size 1.27 1.27)) (justify left bottom))
   )
-  (label "TX1N" (at 144.145 102.235 0)
+  (label "TX1_N" (at 144.145 102.235 0)
     (effects (font (size 1.27 1.27)) (justify left bottom))
   )
@@
     (effects (font (size 1.27 1.27)) (justify left bottom))
   )
-  (label "RX1N" (at 144.145 94.615 0)
+  (label "RX1_N" (at 144.145 94.615 0)
     (effects (font (size 1.27 1.27)) (justify left bottom))
   )
-  (label "RX1P" (at 144.145 97.155 0)
+  (label "RX1_P" (at 144.145 97.155 0)
     (effects (font (size 1.27 1.27)) (justify left bottom))
   )
